File: tester.sch (EAGLE design)
At the start: 76 parts, among them K1 NA, P1 10K, P2 10k lin, Q1 BC847CSMD, Q2 BC847CSMD, Q3 BC847CSMD, Q4 8,000 MHz, Q5 IRL540N, Q6 BC547B, Q7 BC328-40, Q9 IRFU9024, U1 ATmega8/88/168, U2 MCP1702-5002, U3 MCP1702-5002, U4 LM339N

Commit message: history replay r2
Parts:
- removed C111: 100pF, resistor:C-EUC0603
- removed JP7: LCD Display, markus:PINHD-1X16-LCD-TOP
- removed P1: 10K, pot:TRIM_EU-CA6H
- removed Q6: BC547B, transistor-npn:BC547B
- removed Q7: BC328-40, transistor-pnp:BC328-40
- removed R15: 10k, resistor:R-EU_R0603
- removed R18: 10, resistor:R-EU_R0603
- removed R25: 560, resistor:R-EU_R0603
- removed R27: 20, resistor:R-EU_R0603
- removed U$2: 162A, lcd_displays:162A
- added C15: 50u, rcl:CPOL-EUUD-4X5,8
- added DIS1: EA-DOG-M162, ea:EA-DOG-M_LCD
- added M1: SP2000, strapubox:SP2000
- added U$4: (no value), c-infineon_v2:BCR421UHAND
- C13: value 100N -> X7R 10u; device rcl:C-EUC0603K -> rcl:C-EUC0603
- C14, C17: device rcl:C-EUC0603K -> rcl:C-EUC0603
- C6: value 100N -> X7R 1u; device rcl:C-EUC0603K -> rcl:C-EUC0603
- C7: value 2.2µF -> X7R 1u; device rcl:CPOL-EUE5-5 -> rcl:C-EUC0603
- C8: value 2.2µF -> X7R 10u; device rcl:CPOL-EUE5-5 -> rcl:C-EUC0603
- D1: value BAV 103 SMD -> 1N4004
- DC1: value (none) -> 5V/+-15V
- K1: value NA -> NA 05W K
- L1: device rcl:L-EU0204/7 -> EagleLibrary_Wuerth_Elektronik_eiSos_Version_6:WE-RFI_1008
- L2: value 10µH -> L-1008F 33µ; device rcl:L-EU0204/7 -> EagleLibrary_Wuerth_Elektronik_eiSos_Version_6:WE-RFI_1008; CURRENT 0.1A -> (none)
- Q3: value BC847CSMD -> BC328-40; device transistor-npn:BC847CSMD -> transistor-pnp:BC328-40
- Q5: value IRL540N -> BC847CSMD; device transistor-power:IRF3704 -> transistor-npn:BC847CSMD
- Q9: value IRFU9024 -> IRFR9024; device transistor-power:IRFU5305 -> transistor-power:IRFR5305
- U4: value LM339N -> LM339D; device linear:LM339N -> linear:LM339D
- X1: value (none) -> NEB21R; device con-conrad:737992-55 -> con-lumberg:NEB21R
Connections:
- removed net +9V: C5.+, C6.1, C7.+, JP7.A, Q7.C, R11.1, U2.IN, U3.IN
- removed net BL_K: JP7.K, Q5.D
- removed net N$1: P1.A, R15.2
- removed net N$14: Q5.S, R25.2, R27.2
- removed net N$19: C111.1, Q6.B, R25.1
- removed net N$2: JP7.V0, P1.S
- removed net N$26: C13.1, Q9.S, U3.OUT
- new net +5V/2: C13.1, C9.1, DIS1.1, DIS1.20, Q9.S, R19.2, R20.2, R21.2, R22.2, R24.2, U3.OUT, U4P.V+
- new net V+: C15.+, C5.+, C6.1, C7.1, Q3.C, R11.1, U2.IN, U3.IN
- net +30V: now also JP2.5; no longer JP2.4
- net +5V: now also DIS1.23, DIS1.24, DIS1.25, DIS1.26, DIS1.32, DIS1.33, DIS1.34, DIS1.35, DIS1.40, L1.2, Q5.C; no longer C9.1, JP7.VDD, L1.1, Q3.C, R15.1, R19.2, R20.2, R21.2, R22.2, R24.2, U4P.V+
- net GND: now also C15.-, C7.2, C8.2, DIS1.27, DIS1.37, DIS1.38, JP2.4, U$4.GND, X1.1; no longer C7.-, C8.-, JP2.5, JP7.DB0, JP7.DB1, JP7.DB2, JP7.DB3, JP7.R/W, JP7.VSS, P1.E, Q6.E, R27.1, X1.-1
- net N$11: now also X1.3; no longer X1.+
- net N$16: now also U4D.-IN; no longer U4D.+IN
- net N$17: now also U$4.EN; no longer C111.2, Q6.C, R18.1
- net N$18: now also DIS1.19, DIS1.2, U$4.IOUT; no longer Q5.G, R18.2
- net N$20: now also C8.1, L1.1; no longer C8.+, L1.2
- net N$22: now also Q5.B; no longer Q3.B
- net N$23: now also Q5.E; no longer Q3.E
- net N$24: now also L2.1; no longer L2.2
- net N$25: now also L2.2; no longer L2.1
- net N$33: now also Q3.B; no longer Q7.B
- net N$5: now also Q3.E; no longer Q7.E
- net N$6: now also U4D.+IN; no longer U4D.-IN
- net N$9: now also X1.2; no longer X1.K
- net PC0: now also K12.O; no longer K12.P, K13.P
- net PC1: now also K13.O; no longer K12.O
- net PC2: now also K12.P, K13.P; no longer K13.O
- net PD0: now also DIS1.31; no longer JP7.DB4
- net PD1: now also DIS1.30; no longer JP7.DB5
- net PD2: now also DIS1.29; no longer JP7.DB6
- net PD3: now also DIS1.28; no longer JP7.DB7
- net PD4: now also DIS1.39; no longer JP7.RS
- net PD5: now also DIS1.36; no longer JP7.E
Other:
- note removed: "LCD Contrast"
- note removed: "P = 0.6V * I_backlight"
- note removed: "R = 0.6V / I_backlight"
- moved on the sheet: C13, C5, C6, K1, U3, U4D, X1

Commit message: history replay r3
Parts:
- added R18: (no value), pot:TRIM_EU-CA9H
- C5: device rcl:CPOL-EUE5-5 -> rcl:CPOL-EUUD-4X5,8
- D3: device markus:SCHOTTKY-DIODE_RAD3-5-A -> markus:SCHOTTKY-DIODE_3-10
- JP2: value (none) -> TESTSMD
- JP4: value (none) -> TESTZENER; device pinhead:PINHD-1X3 -> pinhead:PINHD-1X4
- U5: value (none) -> BCR421U
- renumbered U$4 to U5
Connections:
- net N$10 renamed AREF
- new net N$1: R18.A, U5.REXT
- net +30V: now also JP4.4
- net GND: now also R18.E, R18.S
- net PC0: now also JP2.3, K12.P, K13.P; no longer JP2.1, K12.O
- net PC1: now also K12.O; no longer K13.O
- net PC2: now also JP2.1, K13.O; no longer JP2.3, K12.P, K13.P

Commit message: history replay r4
Parts:
- L1: CURRENT 0.1A -> (none)
Connections:
- removed net N$20: C8.1, L1.1, U2.OUT
- new net N$2: L1.2, U1.AVCC
- net +5V: now also C8.1, L1.1, U2.OUT; no longer L1.2, U1.AVCC
Other:
- moved on the sheet: L1
Changed lines of the file:
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@@
 <part name="Q3" library="transistor-pnp" deviceset="BC328*" device="" technology="-40"/>
 <part name="D3" library="markus" deviceset="SCHOTTKY-DIODE" device="_3-10" value="SB130"/>
-<part name="L1" library="EagleLibrary_Wuerth_Elektronik_eiSos_Version_6" deviceset="WE-RFI" device="_1008" value="10µH">
-<attribute name="CURRENT" value="0.1A"/>
-</part>
+<part name="L1" library="EagleLibrary_Wuerth_Elektronik_eiSos_Version_6" deviceset="WE-RFI" device="_1008" value="10µH"/>
 <part name="LED1" library="led" deviceset="LED" device="5MM" value="POWER LED"/>
 <part name="G1" library="battery" deviceset="AB9V" device=""/>
@@
 </instance>
 <instance part="D3" gate="G$1" x="60.96" y="208.28"/>
-<instance part="L1" gate="G$1" x="123.19" y="208.28">
-<attribute name="CURRENT" x="120.142" y="201.803" size="1.778" layer="96"/>
-</instance>
+<instance part="L1" gate="G$1" x="171.45" y="190.5"/>
 <instance part="LED1" gate="G$1" x="71.12" y="162.56"/>
 <instance part="G1" gate="G$1" x="53.34" y="193.04" rot="R90"/>
@@
 <wire x1="132.08" y1="208.28" x2="132.08" y2="203.2" width="0.1524" layer="91"/>
 <junction x="132.08" y="208.28"/>
-<pinref part="U1" gate="G$1" pin="AVCC"/>
-<wire x1="180.34" y1="190.5" x2="152.4" y2="190.5" width="0.1524" layer="91"/>
 <pinref part="C3" gate="G$1" pin="2"/>
 <wire x1="152.4" y1="152.4" x2="152.4" y2="190.5" width="0.1524" layer="91"/>
-<junction x="152.4" y="190.5"/>
 <pinref part="R13" gate="G$1" pin="1"/>
+<wire x1="152.4" y1="190.5" x2="152.4" y2="208.28" width="0.1524" layer="91"/>
 <wire x1="160.02" y1="208.28" x2="152.4" y2="208.28" width="0.1524" layer="91"/>
-<wire x1="152.4" y1="208.28" x2="152.4" y2="190.5" width="0.1524" layer="91"/>
 <pinref part="U1" gate="G$1" pin="VCC@1"/>
 <wire x1="180.34" y1="165.1" x2="147.32" y2="165.1" width="0.1524" layer="91"/>
@@
 <wire x1="147.32" y1="165.1" x2="147.32" y2="208.28" width="0.1524" layer="91"/>
 <junction x="147.32" y="208.28"/>
-<pinref part="L1" gate="G$1" pin="2"/>
-<wire x1="128.27" y1="208.28" x2="132.08" y2="208.28" width="0.1524" layer="91"/>
+<pinref part="L1" gate="G$1" pin="1"/>
+<wire x1="166.37" y1="190.5" x2="152.4" y2="190.5" width="0.1524" layer="91"/>
+<junction x="152.4" y="190.5"/>
+<pinref part="U2" gate="IC" pin="OUT"/>
+<wire x1="111.76" y1="208.28" x2="114.3" y2="208.28" width="0.1524" layer="91"/>
+<wire x1="114.3" y1="204.47" x2="114.3" y2="208.28" width="0.1524" layer="91"/>
+<pinref part="C8" gate="G$1" pin="1"/>
+<wire x1="132.08" y1="208.28" x2="114.3" y2="208.28" width="0.1524" layer="91"/>
+<junction x="114.3" y="208.28"/>
 </segment>
 <segment>
@@
 </segment>
 </net>
-<net name="N$20" class="0">
-<segment>
-<pinref part="U2" gate="IC" pin="OUT"/>
-<wire x1="111.76" y1="208.28" x2="114.3" y2="208.28" width="0.1524" layer="91"/>
-<wire x1="114.3" y1="204.47" x2="114.3" y2="208.28" width="0.1524" layer="91"/>
-<pinref part="C8" gate="G$1" pin="1"/>
-<pinref part="L1" gate="G$1" pin="1"/>
-<wire x1="114.3" y1="208.28" x2="118.11" y2="208.28" width="0.1524" layer="91"/>
-<junction x="114.3" y="208.28"/>
-</segment>
-</net>
 <net name="N$21" class="0">
 <segment>
@@
 </segment>
 </net>
+<net name="N$2" class="0">
+<segment>
+<pinref part="L1" gate="G$1" pin="2"/>
+<pinref part="U1" gate="G$1" pin="AVCC"/>
+<wire x1="176.53" y1="190.5" x2="180.34" y2="190.5" width="0.1524" layer="91"/>
+</segment>
+</net>

Commit message: history replay r5
Parts:
- removed L1: 10µH, EagleLibrary_Wuerth_Elektronik_eiSos_Version_6:WE-RFI_1008
- removed M1: SP2000, strapubox:SP2000
- removed U1: ATmega8/88/168, avr-6:MEGA8-P
- added IC1: ATmega8/88/168, avr-7:MEGA8-PU
- added JP5: TESTSMD, pinhead:PINHD-1X5
- added M2: SP2000, strapubox:SP2000
Connections:
- removed net N$2: L1.2, U1.AVCC
- new net TEST1: JP5.1
- new net TEST2: JP5.2
- new net TEST3: JP5.3
- new net TESTZ+: JP5.4
- new net TESTZ-: JP5.5
- net +30V: now also JP2.4; no longer JP2.5
- net +5V: now also IC1.AVCC, IC1.VCC@1; no longer L1.1, U1.VCC@1
- net AREF: now also IC1.AREF; no longer U1.AREF
- net GND: now also IC1.AGND, IC1.GND@1, JP2.5; no longer JP2.4, U1.AGND, U1.GND@1
- net N$12: now also IC1.PB6(XTAL1/TOSC1); no longer U1.PB6(XTAL1/TOSC1)
- net N$13: now also IC1.PB7(XTAL2/TOSC2); no longer U1.PB7(XTAL2/TOSC2)
- net PB0: now also IC1.PB0(ICP1); no longer U1.PB0(ICP)
- net PB1: now also IC1.PB1(OC1A); no longer U1.PB1(OC1A)
- net PB2: now also IC1.PB2(SS/OC1B); no longer U1.PB2(SS/OC1B)
- net PB3: now also IC1.PB3(MOSI/OC2); no longer U1.PB3(MOSI/OC2)
- net PB4: now also IC1.PB4(MISO); no longer U1.PB4(MISO)
- net PB5: now also IC1.PB5(SCK); no longer U1.PB5(SCK)
- net PC0: now also IC1.PC0(ADC0), JP2.1, K13.O; no longer JP2.3, K12.P, K13.P, U1.PC0(ADC0)
- net PC1: now also IC1.PC1(ADC1); no longer U1.PC1(ADC1)
- net PC2: now also IC1.PC2(ADC2), JP2.3, K12.P, K13.P; no longer JP2.1, K13.O, U1.PC2(ADC2)
- net PC3: now also IC1.PC3(ADC3); no longer U1.PC3(ADC3)
- net PC4: now also IC1.PC4(ADC4/SDA); no longer U1.PC4(ADC4/SDA)
- net PC5: now also IC1.PC5(ADC5/SCL); no longer U1.PC5(ADC5/SCL)
- net PC6: now also IC1.PC6(/RESET); no longer U1.PC6(/RESET)
- net PD0: now also IC1.PD0(RXD); no longer U1.PD0(RXD)
- net PD1: now also IC1.PD1(TXD); no longer U1.PD1(TXD)
- net PD2: now also IC1.PD2(INT0); no longer U1.PD2(INT0)
- net PD3: now also IC1.PD3(INT1); no longer U1.PD3(INT1)
- net PD4: now also IC1.PD4(T0/XCK); no longer U1.PD4(XCK/T0)
- net PD5: now also IC1.PD5(T1); no longer U1.PD5(T1)
- net PD6: now also IC1.PD6(AIN0); no longer U1.PD6(AIN0)
- net PD7: now also IC1.PD7(AIN1); no longer U1.PD7(AIN1)
Other:
- note added: ""dreckige" Spannungsversorgung"
- note added: ""saubere" Spannungsversorgung"
- moved on the sheet: C1, C11, C12, C14, C15, C17, C2, C3, C4, C7, C8, D1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

Commit message: history replay r6
Parts:
- removed M2: SP2000, strapubox:SP2000
- removed R18: (no value), pot:TRIM_EU-CA9H
- added JP6: (no value), pinhead:PINHD-1X2
- added M1: SP6000, strapubox:SP6000
- added P1: 250, pot:TRIM_EU-CA6H
- C15, C5: value 50u -> 47u; device rcl:CPOL-EUUD-4X5,8 -> rcl:CPOL-EUUD-5X5,8
- C17: value 10N -> 10n
- C2: value 10nF -> 10n
- D1: value 1N4004 -> BAV 103; device mod_diode:SM4004 -> diode:DIODE-SOD80C
- JP1: value TEST -> ISP; device pinhead:PINHD-1X5 -> con-ml:ML6
- JP2: value TESTSMD -> TEST; device pinhead:PINHD-1X5 -> con-lsta:FE05-1
- JP3: value ISP -> TESTZENER; device con-ml:ML6 -> con-lsta:FE04-1
- JP4: value TESTZENER -> TESTSMD; device pinhead:PINHD-1X4 -> pinhead:PINHD-1X5; REICHELT (none) -> AW 226/20
- JP5: REICHELT (none) -> AW 122/xx
- LED1: device led:LED5MM -> led:LED5MMEXT
- P2: device pot:TRIM_EU-CA6V -> pot:TRIM_EU-S75P
- R3: TOLERANCE 0,1% -> 0.1%
- S1: value 9077-1 -> TOGGLESWITCH; device switch-misc:9077-1 -> external:TOGGLESWITCH
- renumbered U$1 to U1
Connections:
- net +30V: now also JP3.2, JP3.3, JP3.4; no longer JP2.4, JP4.2, JP4.3
- net +5V: now also JP1.2; no longer JP3.2
- net GND: now also JP1.6, JP3.1, JP4.5, P1.E, P1.S; no longer JP2.5, JP3.6, JP4.1, R18.E, R18.S
- net N$1: now also P1.A; no longer R18.A
- net N$21: now also JP6.2; no longer S1.P
- net N$3: now also JP6.1; no longer S1.S
- net PB3: now also JP1.4; no longer JP3.4
- net PB4: now also JP1.1; no longer JP3.1
- net PB5: now also JP1.3; no longer JP3.3
- net PC0: now also JP2.2, JP4.1, K12.O; no longer JP1.1, JP1.2, K13.O
- net PC1: now also JP2.3, JP4.2, K13.O; no longer JP1.3, JP2.2, K12.O
- net PC2: now also JP2.4, JP2.5, JP4.3; no longer JP1.4, JP1.5, JP2.3
- net PC6: now also JP1.5; no longer JP3.5

Commit message: history replay r7
Parts:
- removed JP5: TESTSMD, pinhead:PINHD-1X5
- added PLATINENSAMMLER: LP_NUMBER08_SILK_TOP, Platinensammler:LP_NUMBER08_SILK_TOP
- M1: value SP6000 -> SP6000C-180; device strapubox:SP6000 -> strapubox:SP6000C-180
Connections:
- removed net TEST1: JP5.1
- removed net TEST2: JP5.2
- removed net TEST3: JP5.3
- removed net TESTZ+: JP5.4
- removed net TESTZ-: JP5.5
