File: tester.sch (EAGLE design)
At the start: 76 parts, among them IC1 ATmega8/88/168, K1 NA 05W K, M1 SP6000C-180, P1 250, P2 10k lin, Q1 BC847CSMD, Q2 BC847CSMD, Q3 BC807-40SMD, Q4 8,000 MHz, Q5 BC847CSMD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

Commit message: rotary encoder is PD1 and PD3
Connections:
- net PD1: now also R29.2
- net PD2: no longer R29.2
Changed lines of the file:
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@@
 <pinref part="DIS1" gate="G$1" pin="28"/>
+</segment>
+<segment>
+<pinref part="R29" gate="G$1" pin="2"/>
+<wire x1="215.9" y1="127" x2="215.9" y2="119.38" width="0.1524" layer="91"/>
+<label x="215.9" y="121.92" size="1.778" layer="95" rot="R90"/>
+<wire x1="215.9" y1="127" x2="218.44" y2="129.54" width="0.1524" layer="91"/>
 </segment>
 </net>
@@
 <wire x1="162.56" y1="111.76" x2="162.56" y2="127" width="0.1524" layer="91"/>
 </segment>
-<segment>
-<wire x1="218.44" y1="129.54" x2="215.9" y2="127" width="0.1524" layer="91"/>
-<pinref part="R29" gate="G$1" pin="2"/>
-<wire x1="215.9" y1="127" x2="215.9" y2="119.38" width="0.1524" layer="91"/>
-</segment>
 </net>
 <net name="PD3" class="0">
@@
 <pinref part="R26" gate="G$1" pin="2"/>
 <wire x1="220.98" y1="127" x2="220.98" y2="124.46" width="0.1524" layer="91"/>
+<label x="220.98" y="121.92" size="1.778" layer="95" rot="R90"/>
 </segment>
 </net>
