File: smd-adapter.brd (EAGLE design)
At the start: 19.7 x 26.7 mm, 8 parts

Commit message: shrinked
Parts:
- removed PLATINENSAMMLER: (no value), Platinensammler:LP_NUMBER_BOT
- moved E$6 0.64 mm to (-8.26, 3.81)
Other:
- board size 19.7 x 26.7 mm -> 19.1 x 24.8 mm
Changed lines of the file:
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@@
 <setting verticaltext="up"/>
 </settings>
-<grid distance="0.05" unitdist="inch" unit="mm" style="lines" multiple="1" display="yes" altdistance="0.025" altunitdist="inch" altunit="mm"/>
+<grid distance="0.635" unitdist="mm" unit="mm" style="lines" multiple="1" display="yes" altdistance="5" altunitdist="mil" altunit="mic"/>
 <layers>
 <layer number="1" name="Top" color="4" fill="1" visible="yes" active="yes"/>
@@
 <plain>
 <polygon width="0.254" layer="29">
-<vertex x="1.27" y="25.4"/>
-<vertex x="8.636" y="25.4"/>
+<vertex x="1.27" y="24.765"/>
+<vertex x="8.636" y="24.765"/>
 <vertex x="8.636" y="19.812"/>
 <vertex x="7.874" y="19.812"/>
@@
 </polygon>
 <polygon width="0.254" layer="29">
-<vertex x="9.144" y="25.4"/>
+<vertex x="9.144" y="24.765"/>
 <vertex x="9.144" y="19.812"/>
 <vertex x="9.906" y="19.812"/>
@@
 <vertex x="13.843" y="12.7"/>
 <vertex x="18.415" y="12.7"/>
-<vertex x="18.415" y="25.4"/>
+<vertex x="18.415" y="24.765"/>
 </polygon>
 <polygon width="0.254" layer="29">
@@
 <text x="15.113" y="2.921" size="2" layer="25" ratio="12">Z+</text>
 <text x="1.27" y="2.921" size="2" layer="25" ratio="12">Z-</text>
-<wire x1="0" y1="26.67" x2="19.685" y2="26.67" width="0" layer="20"/>
+<wire x1="0" y1="25.4" x2="19.05" y2="25.4" width="0" layer="20"/>
 <wire x1="4.445" y1="5.715" x2="18.415" y2="5.715" width="0.4064" layer="21"/>
 <polygon width="0.254" layer="29">
@@
 <vertex x="18.415" y="7.747"/>
 </polygon>
-<wire x1="0" y1="26.67" x2="0" y2="0" width="0" layer="20"/>
-<wire x1="0" y1="0" x2="19.685" y2="0" width="0" layer="20"/>
-<wire x1="19.685" y1="0" x2="19.685" y2="26.67" width="0" layer="20"/>
+<wire x1="0" y1="25.4" x2="0" y2="0.635" width="0" layer="20"/>
+<wire x1="0" y1="0.635" x2="19.05" y2="0.635" width="0" layer="20"/>
+<wire x1="19.05" y1="0.635" x2="19.05" y2="25.4" width="0" layer="20"/>
 </plain>
 <attributes>
@@
 </class>
 </classes>
-<designrules name="default">
-<description language="de">&lt;b&gt;EAGLE Design Rules&lt;/b&gt;
+<designrules name="DFRobot_Eagle_Rule_v0.4">
+<description language="en">
+&lt;b&gt;EAGLE Design Rules&lt;/b&gt;
 &lt;p&gt;
-Die Standard-Design-Rules sind so gewählt, dass sie für
-die meisten Anwendungen passen. Sollte ihre Platine
-besondere Anforderungen haben, treffen Sie die erforderlichen
-Einstellungen hier und speichern die Design Rules unter
-einem neuen Namen ab.</description>
-<description language="en">&lt;b&gt;EAGLE Design Rules&lt;/b&gt;
+The default Design Rules have been set to cover
+a wide range of applications. Your particular design
+may have different requirements, so please make the
+necessary adjustments and save your customized
+design rules under a new name.
+</description>
+<description language="it">
+&lt;b&gt;EAGLE Design Rules&lt;/b&gt;
 &lt;p&gt;
 The default Design Rules have been set to cover
@@
 <param name="mtCopper" value="0.035mm 0.035mm 0.035mm 0.035mm 0.035mm 0.035mm 0.035mm 0.035mm 0.035mm 0.035mm 0.035mm 0.035mm 0.035mm 0.035mm 0.035mm 0.035mm"/>
 <param name="mtIsolate" value="1.5mm 0.15mm 0.2mm 0.15mm 0.2mm 0.15mm 0.2mm 0.15mm 0.2mm 0.15mm 0.2mm 0.15mm 0.2mm 0.15mm 0.2mm"/>
-<param name="mdWireWire" value="8mil"/>
-<param name="mdWirePad" value="8mil"/>
-<param name="mdWireVia" value="8mil"/>
-<param name="mdPadPad" value="8mil"/>
-<param name="mdPadVia" value="8mil"/>
-<param name="mdViaVia" value="8mil"/>
-<param name="mdSmdPad" value="8mil"/>
-<param name="mdSmdVia" value="8mil"/>
-<param name="mdSmdSmd" value="8mil"/>
+<param name="mdWireWire" value="6mil"/>
+<param name="mdWirePad" value="6mil"/>
+<param name="mdWireVia" value="6mil"/>
+<param name="mdPadPad" value="6mil"/>
+<param name="mdPadVia" value="6mil"/>
+<param name="mdViaVia" value="6mil"/>
+<param name="mdSmdPad" value="0mil"/>
+<param name="mdSmdVia" value="0mil"/>
+<param name="mdSmdSmd" value="0mil"/>
 <param name="mdViaViaSameLayer" value="8mil"/>
 <param name="mnLayersViaInSmd" value="2"/>
-<param name="mdCopperDimension" value="40mil"/>
-<param name="mdDrill" value="8mil"/>
+<param name="mdCopperDimension" value="10mil"/>
+<param name="mdDrill" value="10mil"/>
 <param name="mdSmdStop" value="0mil"/>
-<param name="msWidth" value="10mil"/>
-<param name="msDrill" value="24mil"/>
-<param name="msMicroVia" value="9.99mm"/>
+<param name="msWidth" value="6mil"/>
+<param name="msDrill" value="12mil"/>
+<param name="msMicroVia" value="12mil"/>
 <param name="msBlindViaRatio" value="0.5"/>
 <param name="rvPadTop" value="0.25"/>
@@
 <param name="rvMicroViaOuter" value="0.25"/>
 <param name="rvMicroViaInner" value="0.25"/>
-<param name="rlMinPadTop" value="10mil"/>
+<param name="rlMinPadTop" value="12mil"/>
 <param name="rlMaxPadTop" value="20mil"/>
 <param name="rlMinPadInner" value="10mil"/>
 <param name="rlMaxPadInner" value="20mil"/>
-<param name="rlMinPadBottom" value="10mil"/>
+<param name="rlMinPadBottom" value="12mil"/>
 <param name="rlMaxPadBottom" value="20mil"/>
 <param name="rlMinViaOuter" value="8mil"/>
@@
 <param name="mvStopFrame" value="1"/>
 <param name="mvCreamFrame" value="0"/>
-<param name="mlMinStopFrame" value="4mil"/>
-<param name="mlMaxStopFrame" value="4mil"/>
+<param name="mlMinStopFrame" value="2mil"/>
+<param name="mlMaxStopFrame" value="2mil"/>
 <param name="mlMinCreamFrame" value="0mil"/>
 <param name="mlMaxCreamFrame" value="0mil"/>
-<param name="mlViaStopLimit" value="0mil"/>
+<param name="mlViaStopLimit" value="25mil"/>
 <param name="srRoundness" value="0"/>
 <param name="srMinRoundness" value="0mil"/>
@@
 <elements>
 <element name="JP5" library="pinhead" package="1X05" value="TESTSMD" x="2.54" y="11.43" smashed="yes" rot="MR270">
-<attribute name="VALUE" x="5.715" y="17.78" size="1.27" layer="28" rot="MR270"/>
 <attribute name="REICHELT" value="AW 122/xx" x="2.54" y="11.43" size="1.778" layer="28" rot="MR270" display="off"/>
 </element>
@@
 <attribute name="VALUE" x="-4.67" y="22.394" size="1.27" layer="27" rot="R180"/>
 </element>
-<element name="E$6" library="ref-packages" package="MELF-MLL41" value="" x="-8.255" y="3.175" smashed="yes">
-<attribute name="VALUE" x="-10.795" y="0" size="1.27" layer="27"/>
-</element>
-<element name="PLATINENSAMMLER" library="Platinensammler" package="LP_NUMBER_BOT" value="" x="15.24" y="24.13"/>
+<element name="E$6" library="ref-packages" package="MELF-MLL41" value="" x="-8.255" y="3.81" smashed="yes">
+<attribute name="VALUE" x="-10.795" y="0.635" size="1.27" layer="27"/>
+</element>
 </elements>
 <signals>
@@
 <vertex x="9.906" y="19.812"/>
 <vertex x="9.144" y="19.812"/>
-<vertex x="9.144" y="25.4"/>
-<vertex x="18.415" y="25.4"/>
+<vertex x="9.144" y="24.765"/>
+<vertex x="18.415" y="24.765"/>
 <vertex x="18.415" y="12.7"/>
 <vertex x="13.843" y="12.7"/>
@@
 <vertex x="7.874" y="19.812"/>
 <vertex x="8.636" y="19.812"/>
-<vertex x="8.636" y="25.4"/>
-<vertex x="1.27" y="25.4"/>
+<vertex x="8.636" y="24.765"/>
+<vertex x="1.27" y="24.765"/>
 </polygon>
 </signal>
